Commit message: Add camera adapter

File: xarm_description/urdf/xarm_device.urdf.xacro (robot description, xacro)
@@ -19,4 +19,9 @@
   <xacro:arg name="add_realsense_d435i" default="false"/>
   <xacro:arg name="add_d435i_links" default="true"/>
+  <xacro:arg name="add_camera_adapter" default="false"/>
+  <xacro:arg name="camera_adapter_xyz" default="0 0 0"/>
+  <xacro:arg name="camera_adapter_rpy" default="0 0 0"/>
+  <xacro:arg name="camera_adapter_tool_xyz" default="0 0 0.0015"/>
+  <xacro:arg name="camera_adapter_tool_rpy" default="0 0 0"/>
   <xacro:arg name="use_gazebo_camera" default="false"/>
   <xacro:arg name="add_other_geometry" default="false"/>
@@ -49,4 +54,9 @@
     add_realsense_d435i="$(arg add_realsense_d435i)"
     add_d435i_links="$(arg add_d435i_links)"
+    add_camera_adapter="$(arg add_camera_adapter)"
+    camera_adapter_xyz="$(arg camera_adapter_xyz)"
+    camera_adapter_rpy="$(arg camera_adapter_rpy)"
+    camera_adapter_tool_xyz="$(arg camera_adapter_tool_xyz)"
+    camera_adapter_tool_rpy="$(arg camera_adapter_tool_rpy)"
     add_other_geometry="$(arg add_other_geometry)"
     geometry_type="$(arg geometry_type)" geometry_mass="$(arg geometry_mass)"

File: xarm_description/urdf/xarm_device_macro.xacro (robot description, xacro)
@@ -21,4 +21,9 @@
     add_realsense_d435i:=false
     add_d435i_links:=true
+    add_camera_adapter:=false
+    camera_adapter_xyz:='0 0 0'
+    camera_adapter_rpy:='0 0 0'
+    camera_adapter_tool_xyz:='0 0 0.0015'
+    camera_adapter_tool_rpy:='0 0 0'
     use_gazebo_camera:=false
     add_other_geometry:=false
@@ -226,14 +231,25 @@
       <child link="${prefix}link_eef" />
     </joint>
+    <xacro:property name="tool_attach_link" value="${prefix}link_eef"/>
+    <xacro:property name="tool_attach_xyz" value="0 0 0"/>
+    <xacro:property name="tool_attach_rpy" value="0 0 0"/>
+    <xacro:if value="${add_camera_adapter}">
+      <xacro:include filename="$(find xarm_description)/urdf/end_tool/camera_adapter.urdf.xacro" />
+      <xacro:camera_adapter_urdf prefix="${prefix}" attach_to="${prefix}link_eef"
+        attach_xyz="${camera_adapter_xyz}" attach_rpy="${camera_adapter_rpy}" />
+      <xacro:property name="tool_attach_link" value="${prefix}camera_adapter_link"/>
+      <xacro:property name="tool_attach_xyz" value="${camera_adapter_tool_xyz}"/>
+      <xacro:property name="tool_attach_rpy" value="${camera_adapter_tool_rpy}"/>
+    </xacro:if>
     <xacro:if value="${add_gripper}">
       <xacro:if value="${robot_type == 'lite'}">
         <!-- Load Lite Gripper Model URDF -->
         <xacro:include filename="$(find xarm_description)/urdf/gripper/lite_gripper.urdf.xacro" />
-        <xacro:uflite_gripper_urdf prefix="${prefix}" attach_to="${prefix}link_eef" />
+        <xacro:uflite_gripper_urdf prefix="${prefix}" attach_to="${tool_attach_link}" attach_xyz="${tool_attach_xyz}" attach_rpy="${tool_attach_rpy}" />
       </xacro:if>
       <xacro:unless value="${robot_type == 'lite'}">
         <!-- Load XArm Gripper Model URDF -->
         <xacro:include filename="$(find xarm_description)/urdf/gripper/xarm_gripper_macro.xacro" />
-        <xacro:xarm_gripper_macro prefix="${prefix}" attach_to="${prefix}link_eef"
+        <xacro:xarm_gripper_macro prefix="${prefix}" attach_to="${tool_attach_link}" attach_xyz="${tool_attach_xyz}" attach_rpy="${tool_attach_rpy}"
           ros2_control_plugin="${ros2_control_plugin}" dof="${dof}" hard_interface="${hard_interface}" />
       </xacro:unless>
@@ -243,5 +259,5 @@
         <!-- Load BIO Gripper Model URDF -->
         <xacro:include filename="$(find xarm_description)/urdf/gripper/bio_gripper_macro.xacro" />
-        <xacro:bio_gripper_macro prefix="${prefix}" attach_to="${prefix}link_eef"
+        <xacro:bio_gripper_macro prefix="${prefix}" attach_to="${tool_attach_link}" attach_xyz="${tool_attach_xyz}" attach_rpy="${tool_attach_rpy}"
           ros2_control_plugin="${ros2_control_plugin}" dof="${dof}" hard_interface="${hard_interface}" />
       </xacro:unless>
@@ -251,10 +267,10 @@
         <!-- Load Lite Vacuum Gripper Model URDF -->
         <xacro:include filename="$(find xarm_description)/urdf/vacuum_gripper/lite_vacuum_gripper.urdf.xacro" />
-        <xacro:uflite_vacuum_gripper_urdf prefix="${prefix}" attach_to="${prefix}link_eef" />
+        <xacro:uflite_vacuum_gripper_urdf prefix="${prefix}" attach_to="${tool_attach_link}" attach_xyz="${tool_attach_xyz}" attach_rpy="${tool_attach_rpy}" />
       </xacro:if>
       <xacro:unless value="${robot_type == 'lite'}">
         <!-- Load XArm Vacuum Gripper Model URDF -->
         <xacro:include filename="$(find xarm_description)/urdf/vacuum_gripper/xarm_vacuum_gripper.urdf.xacro" />
-        <xacro:xarm_vacuum_gripper_urdf prefix="${prefix}" attach_to="${prefix}link_eef" />
+        <xacro:xarm_vacuum_gripper_urdf prefix="${prefix}" attach_to="${tool_attach_link}" attach_xyz="${tool_attach_xyz}" attach_rpy="${tool_attach_rpy}" />
       </xacro:unless>
     </xacro:if>
@@ -262,5 +278,5 @@
       <!-- Load Other Model URDF -->
       <xacro:include filename="$(find xarm_description)/urdf/other/other_geometry.urdf.xacro" />
-      <xacro:other_geometry prefix="${prefix}" attach_to="${prefix}link_eef"
+      <xacro:other_geometry prefix="${prefix}" attach_to="${tool_attach_link}" attach_xyz="${tool_attach_xyz}" attach_rpy="${tool_attach_rpy}"
         geometry_type="${geometry_type}" geometry_mass="${geometry_mass}"
         geometry_height="${geometry_height}" geometry_radius="${geometry_radius}"
